Commit message: Rebuild RobotModel and Give Drive Control

File: description/robot_core.xacro (robot description, xacro)
@@ -2,4 +2,13 @@
 <robot xmlns:xacro="http://www.ros.org/wiki/xacro">
     <xacro:include filename="inertial_macros.xacro"/>
+    <xacro:include filename="vertical_post.xacro"/>
+    <!-- Left Cylinder-->
+    <xacro:vertical_post name="post1" x="0.075" y="-0.099" z="-0.123" color="black"/>
+    <xacro:vertical_post name="post2" x="0.150" y="-0.099" z="-0.123" color="blue"/>
+    <xacro:vertical_post name="post3" x="0.225" y="-0.099" z="-0.123" color="orange"/>
+    <!-- Right Cylinder-->
+    <xacro:vertical_post name="post4" x="0.075" y="0.099" z="-0.123" color="red"/>
+    <xacro:vertical_post name="post5" x="0.150" y="0.099" z="-0.123" color="blue"/>
+    <xacro:vertical_post name="post6" x="0.225" y="0.099" z="-0.123" color="white"/>
     <material name="white">
         <color rgba="1 1 1 1"/>
@@ -13,4 +22,7 @@
     <material name="black">
         <color rgba="0 0 0 1"/>
+    </material>
+    <material name="red">
+        <color rgba="1.0 0.0 0.0 1.0"/>
     </material>
     <!-- Base Link-->
@@ -27,5 +39,5 @@
             <origin xyz="0.15 0 0.075"/>
             <geometry>
-                <box size="0.3 0.3 0.15"/>
+                <box size="0.2 0.3 0.035"/>
             </geometry>
             <material name="white">
@@ -35,16 +47,35 @@
             <origin xyz="0.15 0 0.075"/>
             <geometry>
-                <box size="0.3 0.3 0.15"/>
+                <box size="0.2 0.3 0.035"/>
             </geometry>
         </collision>
-        <xacro:inertial_box mass="0.5" x="0.3" y="0.3" z="0.15">
+        <xacro:inertial_box mass="0.1" x="0.2" y="0.3" z="0.035">
             <origin xyz="0.15 0.0 0.075" rpy="0.0 0.0 0.0"/>
         </xacro:inertial_box>
+        <visual>
+            <origin xyz="0.15 0.0 -0.005"/>
+            <geometry>
+                <box size="0.2 0.3 0.035"/>
+            </geometry>
+            <material name="white">
+            </material>
+        </visual>
+        <collision>
+            <origin xyz="0.15 0.0 -0.005"/>
+            <geometry>
+                <box size="0.2 0.3 0.035"/>
+            </geometry>
+        </collision>
     </link>
+    <gazebo reference="chassis">
+        <material>
+            Gazebo/White
+        </material>
+    </gazebo>
     <!-- Left Wheel link-->
      <joint name="left_wheel_link" type="continuous">
         <parent link="base_link"/>
         <child link="left_wheel"/>
-        <origin xyz = "0 0.175 0" rpy="-${pi/2} 0.0 0.0"/>
+        <origin xyz = "0 0.165 0" rpy="-${pi/2} 0.0 0.0"/>
         <axis xyz="0.0 0.0 1"/>
      </joint>
@@ -52,5 +83,5 @@
         <visual>
             <geometry>
-                <cylinder radius="0.05" length="0.04"/>
+                <cylinder radius="0.04" length="0.03"/>
             </geometry>
             <material name="blue">
@@ -59,16 +90,21 @@
            <collision>
             <geometry>
-                <cylinder radius="0.05" length="0.04"/>
+                <cylinder radius="0.04" length="0.03"/>
             </geometry>
         </collision>
-        <xacro:inertial_cylinder mass="0.1" length="0.04" radius="0.05">
+        <xacro:inertial_cylinder mass="0.1" length="0.03" radius="0.04">
             <origin xyz="0.0 0.0 0.0" rpy="0.0 0.0 0.0"/>
         </xacro:inertial_cylinder>
      </link>
+      <gazebo reference="left_wheel">
+        <material>
+            Gazebo/Blue
+        </material>
+    </gazebo>
      <!-- Right Wheel link-->
      <joint name="right_wheel_link" type="continuous">
         <parent link="base_link"/>
         <child link="right_wheel"/>
-        <origin xyz = "0 -0.175 0" rpy="${pi/2} 0.0 0.0"/>
+        <origin xyz = "0 -0.165 0" rpy="${pi/2} 0.0 0.0"/>
         <axis xyz="0.0 0.0 -1"/>
      </joint>
@@ -76,5 +112,5 @@
         <visual>
             <geometry>
-                <cylinder radius="0.05" length="0.04"/>
+                <cylinder radius="0.04" length="0.03"/>
             </geometry>
             <material name="blue">
@@ -83,21 +119,26 @@
         <collision>
             <geometry>
-                <cylinder radius="0.05" length="0.04"/>
+                <cylinder radius="0.04" length="0.03"/>
             </geometry>
         </collision>
-        <xacro:inertial_cylinder mass="0.1" length="0.04" radius="0.05">
+        <xacro:inertial_cylinder mass="0.1" length="0.03" radius="0.04">
             <origin xyz="0.0 0.0 0.0" rpy="0.0 0.0 0.0"/>
         </xacro:inertial_cylinder>
      </link>
+      <gazebo reference="right_wheel">
+        <material>
+            Gazebo/Blue
+        </material>
+    </gazebo>
      <!-- Caster Wheel Link-->
       <joint name ="caster_wheel_link" type = "fixed">
         <parent link="chassis"/>
         <child link="caster_wheel"/>
-        <origin xyz = "0.24 0 0"/>
+        <origin xyz = "0.23 0 -0.02"/>
       </joint>
       <link name="caster_wheel">
         <visual>
             <geometry>
-                <sphere radius="0.05"/>
+                <sphere radius="0.02"/>
             </geometry>
             <material name="black">
@@ -106,10 +147,17 @@
            <collision>
             <geometry>
-                <sphere radius="0.05"/>
+                <sphere radius="0.02"/>
             </geometry>
         </collision>
-        <xacro:inertial_sphere mass="0.1" radius="0.05">
+        <xacro:inertial_sphere mass="0.1" radius="0.02">
             <origin xyz="0.0 0.0 0.0" rpy="0.0 0.0 0.0"/>
         </xacro:inertial_sphere>
       </link>
+       <gazebo reference="caster_wheel">
+        <material>
+            Gazebo/Black
+        </material>
+        <mu1 value="0.001"></mu1>
+        <mu2 value="0.001"></mu2>
+    </gazebo>
 </robot>
