Commit message: Fix Size Of Verticla post

File: description/vertical_post.xacro (robot description, xacro)
@@ -7,5 +7,5 @@
                 <mass value="0.001"/>
                 <geometry>
-                    <cylinder length="0.08" radius="0.01"/>
+                    <cylinder length="0.08" radius="0.005"/>
                 </geometry>
                 <material name="${color}"/>
@@ -14,5 +14,5 @@
                 <origin xyz="0 0 0.15"/>
                 <geometry>
-                    <cylinder length="0.08" radius="0.01"/>
+                    <cylinder length="0.08" radius="0.005"/>
                 </geometry>
             </collision>
