Commit message: Update

File: description/gazebo_control.xacro (robot description, xacro)
@@ -4,6 +4,6 @@
         <plugin name="diff_drive" filename="libgazebo_ros_diff_drive.so">
             <!-- Wheel Information -->
-            <left_joint>left_wheel_joint</left_joint>
-            <right_joint>right_wheel_joint</right_joint>
+            <left_joint>left_wheel_link</left_joint>
+            <right_joint>right_wheel_link</right_joint>
             <wheel_separation>0.297</wheel_separation>
             <wheel_diameter>0.066</wheel_diameter>

File: description/robot_core.xacro (robot description, xacro)
@@ -150,5 +150,5 @@
             </geometry>
         </collision>
-        <xacro:inertial_sphere mass="0.1" radius="0.02">
+        <xacro:inertial_sphere mass="1" radius="0.02">
             <origin xyz="0.0 0.0 0.0" rpy="0.0 0.0 0.0"/>
         </xacro:inertial_sphere>
@@ -158,6 +158,6 @@
             Gazebo/Black
         </material>
-        <mu1 value="0.001"></mu1>
-        <mu2 value="0.001"></mu2>
+        <mu1 value="0.1"></mu1>
+        <mu2 value="0.1"></mu2>
     </gazebo>
 </robot>

File: description/vertical_post.xacro (robot description, xacro)
@@ -5,7 +5,7 @@
             <visual>
                 <origin xyz="0 0 0.15"/>
+                <mass value="0.001"/>
                 <geometry>
                     <cylinder length="0.08" radius="0.01"/>
-                    <mass value="0.01"/>
                 </geometry>
                 <material name="${color}"/>

Commit message: Config all file

File: description/gazebo_control.xacro (robot description, xacro)
@@ -4,6 +4,6 @@
         <plugin name="diff_drive" filename="libgazebo_ros_diff_drive.so">
             <!-- Wheel Information -->
-            <left_joint>left_wheel_link</left_joint>
-            <right_joint>right_wheel_link</right_joint>
+            <left_joint>left_wheel_joint</left_joint>
+            <right_joint>right_wheel_joint</right_joint>
             <wheel_separation>0.297</wheel_separation>
             <wheel_diameter>0.066</wheel_diameter>

File: description/lidar.xacro (robot description, xacro)
@@ -1,22 +1,29 @@
 <?xml version="1.0"?>
-<robot xmlns:xacro="http://www.ros.org/wiki/xacro" >
+<robot xmlns:xacro="http://www.ros.org/wiki/xacro"  name="robot">
     <joint name="laser_joint" type="fixed">
         <parent link="chassis"/>
-        <child link="laser_frame"/>
-        <origin xyz="0.1 0 0.089" rpy="0 0 0"/>
+        <child link="laser"/>
+        <origin xyz="0.22 0 0.15" rpy="0 0 ${pi}"/>
     </joint>
-    <link name="laser_frame">
+    <link name="laser">
         <visual>
             <geometry>
-                <cylinder radius="0.02" length="0.03"/>
+                <cylinder radius="0.025" length="0.02"/>
             </geometry>
-            <material name="red"/>
+            <material name="black"/>
+        </visual>
+        <visual>
+            <origin xyz="0 0 -0.02"/>
+            <geometry>
+                <box size="0.05 0.05 0.02"/>
+            </geometry>
+            <material name="black"/>
         </visual>
         <collision>
             <geometry>
-                <cylinder radius="0.02" length="0.03"/>
+                <cylinder radius="0.025" length="0.02"/>
             </geometry>
         </collision>
-        <xacro:inertial_cylinder mass="0.1" length="0.03" radius="0.02">
+        <xacro:inertial_cylinder mass="0.1" length="0.02" radius="0.025">
             <origin xyz="0 0 0" rpy="0 0 0"/>
         </xacro:inertial_cylinder>
@@ -25,11 +32,12 @@
         <material>Gazebo/Red</material>
         <sensor name="laser" type="ray">
-            <pose> 0 0 0 0 0 0 </pose>
-            <visualize>true</visualize>
+            <pose> 0 0 0 0</pose>
+            <visualize>false</visualize>
             <update_rate>10</update_rate>
             <ray>
                 <scan>
                     <horizontal>
-                        <samples>360</samples>
+                        <sample>360</sample>
+                        <resolution>1</resolution>
                         <min_angle>-3.14</min_angle>
                         <max_angle>3.14</max_angle>
@@ -38,5 +46,6 @@
                 <range>
                     <min>0.3</min>
-                    <max>12</max>
+                    <max>5</max>
+                    <resolution>0.01</resolution>
                 </range>
             </ray>

File: description/robot.urdf.xacro (robot description, xacro)
@@ -1,16 +1,16 @@
 <?xml version="1.0"?>
 <robot xmlns:xacro="http://www.ros.org/wiki/xacro"  name="robot">
-<!--
     <xacro:arg name="use_ros2_control" default="true"/>
-    <xacro:arg name="sim_node" default="false"/>
+    <xacro:arg name="sim_mode" default="false"/>
+    <xacro:include filename="robot_core.xacro" />
     <xacro:if value="$(arg use_ros2_control)">
-        <xacro:include filename="ros2_control.xacro"/>
-    </xacro:if> -->
-    <!-- <xacro:unless value="$(use_ros2_control)">
-        <xacro:include filename="gazebo_control.xacro"/>
-    </xacro:unless> -->
-    <xacro:include filename="robot_core.xacro"/>
-    <xacro:include filename="gazebo_control.xacro"/>
-    <xacro:include filename="lidar.xacro"/>
-    <xacro:include filename="camera.xacro"/>
+        <xacro:include filename="ros2_control.xacro" />
+    </xacro:if>
+    <xacro:unless value="$(arg use_ros2_control)">
+        <xacro:include filename="gazebo_control.xacro" />
+    </xacro:unless>
+    <xacro:include filename="lidar.xacro" />
+    <!-- <xacro:include filename="camera.xacro" /> -->
+    <!-- <xacro:include filename="depth_camera.xacro" /> -->
+    <!-- <xacro:include filename="face.xacro" /> -->
 </robot>

File: description/robot_core.xacro (robot description, xacro)
@@ -2,13 +2,4 @@
 <robot xmlns:xacro="http://www.ros.org/wiki/xacro">
     <xacro:include filename="inertial_macros.xacro"/>
-    <xacro:include filename="vertical_post.xacro"/>
-    <!-- Left Cylinder-->
-    <xacro:vertical_post name="post1" x="0.075" y="-0.099" z="-0.123" color="black"/>
-    <xacro:vertical_post name="post2" x="0.150" y="-0.099" z="-0.123" color="blue"/>
-    <xacro:vertical_post name="post3" x="0.225" y="-0.099" z="-0.123" color="orange"/>
-    <!-- Right Cylinder-->
-    <xacro:vertical_post name="post4" x="0.075" y="0.099" z="-0.123" color="red"/>
-    <xacro:vertical_post name="post5" x="0.150" y="0.099" z="-0.123" color="blue"/>
-    <xacro:vertical_post name="post6" x="0.225" y="0.099" z="-0.123" color="white"/>
     <material name="white">
         <color rgba="1 1 1 1"/>
@@ -20,144 +11,140 @@
         <color rgba="0.2 0.2 1 1"/>
     </material>
+    <material name="red">
+        <color rgba="1 0 0 1"/>
+    </material>
     <material name="black">
         <color rgba="0 0 0 1"/>
     </material>
-    <material name="red">
-        <color rgba="1.0 0.0 0.0 1.0"/>
-    </material>
-    <!-- Base Link-->
+    <!-- BASE LINK -->
     <link name="base_link">
     </link>
+    <!-- BASE_FOOTPRINT_LINK -->
+    <joint name="base_footprint_joint" type="fixed">
+        <parent link="base_link"/>
+        <child link="base_footprint"/>
+        <origin xyz="0 0 0" rpy="0 0 0"/>
+    </joint>
+    <link name="base_footprint">
+    </link>
+    <!-- CHASSIS LINK -->
     <joint name="chassis_joint" type="fixed">
         <parent link="base_link"/>
         <child link="chassis"/>
-        <origin xyz="-0.1 0.0 0.0"/>
+        <origin xyz="-0.1 0 0"/>
     </joint>
-    <!-- Chassis Link-->
-    <link name ="chassis">
+    <link name="chassis">
         <visual>
-            <origin xyz="0.15 0 0.075"/>
+            <origin xyz="0.17 0 0.0925"/>
             <geometry>
-                <box size="0.2 0.3 0.035"/>
+                <box size="0.2 0.17 0.055"/>
             </geometry>
-            <material name="white">
-            </material>
+            <material name="white"/>
         </visual>
         <collision>
-            <origin xyz="0.15 0 0.075"/>
+            <origin xyz="0.17 0 0.0925"/>
             <geometry>
-                <box size="0.2 0.3 0.035"/>
+                <box size="0.2 0.17 0.055"/>
             </geometry>
         </collision>
-        <xacro:inertial_box mass="0.1" x="0.2" y="0.3" z="0.035">
-            <origin xyz="0.15 0.0 0.075" rpy="0.0 0.0 0.0"/>
+        <xacro:inertial_box mass="0.5" x="0.2" y="0.17" z="0.1">
+            <origin xyz="0.17 0 0.0925" rpy="0 0 0"/>
         </xacro:inertial_box>
-        <visual>
-            <origin xyz="0.15 0.0 -0.005"/>
-            <geometry>
-                <box size="0.2 0.3 0.035"/>
-            </geometry>
-            <material name="white">
-            </material>
-        </visual>
-        <collision>
-            <origin xyz="0.15 0.0 -0.005"/>
-            <geometry>
-                <box size="0.2 0.3 0.035"/>
-            </geometry>
-        </collision>
     </link>
     <gazebo reference="chassis">
-        <material>
-            Gazebo/White
-        </material>
+        <material>Gazebo/Orange</material>
     </gazebo>
-    <!-- Left Wheel link-->
-     <joint name="left_wheel_link" type="continuous">
+    <!-- LEFT WHEEL LINK -->
+    <joint name="left_wheel_joint" type="continuous">
         <parent link="base_link"/>
         <child link="left_wheel"/>
-        <origin xyz = "0 0.165 0" rpy="-${pi/2} 0.0 0.0"/>
-        <axis xyz="0.0 0.0 1"/>
-     </joint>
-     <link name="left_wheel">
+        <origin xyz="0.0175 0.1 0.0325" rpy="-${pi/2} 0 0"/>
+        <axis xyz="0 0 1"/>
+    </joint>
+    <link name="left_wheel">
         <visual>
             <geometry>
-                <cylinder radius="0.04" length="0.03"/>
+                <cylinder radius="0.0325" length="0.027"/>
             </geometry>
-            <material name="blue">
-            </material>
-        </visual>
-           <collision>
-            <geometry>
-                <cylinder radius="0.04" length="0.03"/>
-            </geometry>
-        </collision>
-        <xacro:inertial_cylinder mass="0.1" length="0.03" radius="0.04">
-            <origin xyz="0.0 0.0 0.0" rpy="0.0 0.0 0.0"/>
-        </xacro:inertial_cylinder>
-     </link>
-      <gazebo reference="left_wheel">
-        <material>
-            Gazebo/Blue
-        </material>
-    </gazebo>
-     <!-- Right Wheel link-->
-     <joint name="right_wheel_link" type="continuous">
-        <parent link="base_link"/>
-        <child link="right_wheel"/>
-        <origin xyz = "0 -0.165 0" rpy="${pi/2} 0.0 0.0"/>
-        <axis xyz="0.0 0.0 -1"/>
-     </joint>
-     <link name="right_wheel">
-        <visual>
-            <geometry>
-                <cylinder radius="0.04" length="0.03"/>
-            </geometry>
-            <material name="blue">
-            </material>
+            <material name="blue"/>
         </visual>
         <collision>
             <geometry>
-                <cylinder radius="0.04" length="0.03"/>
+                <cylinder radius="0.0325" length="0.027"/>
             </geometry>
         </collision>
-        <xacro:inertial_cylinder mass="0.1" length="0.03" radius="0.04">
-            <origin xyz="0.0 0.0 0.0" rpy="0.0 0.0 0.0"/>
+        <xacro:inertial_cylinder mass="0.1" length="0.027" radius="0.0325">
+            <origin xyz="0 0 0" rpy="0 0 0"/>
         </xacro:inertial_cylinder>
-     </link>
-      <gazebo reference="right_wheel">
-        <material>
-            Gazebo/Blue
-        </material>
+    </link>
+    <gazebo reference="left_wheel">
+        <material>Gazebo/Blue</material>
     </gazebo>
-     <!-- Caster Wheel Link-->
-      <joint name ="caster_wheel_link" type = "fixed">
+    <!-- RIGHT WHEEL LINK -->
+    <joint name="right_wheel_joint" type="continuous">
+        <parent link="base_link"/>
+        <child link="right_wheel"/>
+        <origin xyz="0.0175 -0.1 0.0325" rpy="${pi/2} 0 0"/>
+        <axis xyz="0 0 -1"/>
+    </joint>
+    <link name="right_wheel">
+        <visual>
+            <geometry>
+                <cylinder radius="0.0325" length="0.027"/>
+            </geometry>
+            <material name="blue"/>
+        </visual>
+        <collision>
+            <geometry>
+                <cylinder radius="0.0325" length="0.027"/>
+            </geometry>
+        </collision>
+        <xacro:inertial_cylinder mass="0.1" length="0.027" radius="0.0325">
+            <origin xyz="0 0 0" rpy="0 0 0"/>
+        </xacro:inertial_cylinder>
+    </link>
+    <gazebo reference="right_wheel">
+        <material>Gazebo/Blue</material>
+    </gazebo>
+    <!-- CASTER WHEEL LINK -->
+    <joint name="caster_wheel_joint" type="fixed">
         <parent link="chassis"/>
         <child link="caster_wheel"/>
-        <origin xyz = "0.23 0 -0.02"/>
-      </joint>
-      <link name="caster_wheel">
+        <origin xyz="0.225 0 0.0325"/>
+    </joint>
+    <link name="caster_wheel">
         <visual>
             <geometry>
-                <sphere radius="0.02"/>
+                <sphere radius="0.0325"/>
             </geometry>
-            <material name="black">
-            </material>
+            <material name="white"/>
         </visual>
-           <collision>
+        <collision>
             <geometry>
-                <sphere radius="0.02"/>
+                <sphere radius="0.0325"/>
             </geometry>
         </collision>
-        <xacro:inertial_sphere mass="1" radius="0.02">
-            <origin xyz="0.0 0.0 0.0" rpy="0.0 0.0 0.0"/>
+        <xacro:inertial_sphere mass="0.1" radius="0.0325">
+            <origin xyz="0 0 0" rpy="0 0 0"/>
         </xacro:inertial_sphere>
-      </link>
-       <gazebo reference="caster_wheel">
-        <material>
-            Gazebo/Black
-        </material>
-        <mu1 value="0.1"></mu1>
-        <mu2 value="0.1"></mu2>
+    </link>
+    <gazebo reference="caster_wheel">
+        <material>Gazebo/Black</material>
+        <mu1 value="0.001"/>
+        <mu2 value="0.001"/>
     </gazebo>
+    <!-- เพิ่ม IMU link ใน URDF -->
+    <link name="imu_link">
+    <visual>
+        <geometry>
+        <box size="0.02 0.02 0.01"/>
+        </geometry>
+        <material name="red"/>
+    </visual>
+    </link>
+    <joint name="imu_joint" type="fixed">
+    <parent link="chassis"/>
+    <child link="imu_link"/>
+    <origin xyz="0.15 0 0.095" rpy="0 0 0"/>
+    </joint>
 </robot>

File: description/ros2_control.xacro (robot description, xacro)
@@ -1,15 +1,57 @@
 <?xml version="1.0"?>
 <robot xmlns:xacro="http://www.ros.org/wiki/xacro">
-    <xacro:unless value="$(arg sim_node)">
+    <xacro:unless value="$(arg sim_mode)">
         <ros2_control name="RealRobot" type="system">
             <hardware>
-                <plugin>diffdrive_arduino/DriffDriveArduino</plugin>
+                <plugin>diffdrive_arduino/DiffDriveArduino</plugin>
                 <param name="left_wheel_name">left_wheel_joint</param>
                 <param name="right_wheel_name">right_wheel_joint</param>
                 <param name="loop_rate">30</param>
-                <param name="device">/dev/ttyUSB0</param>
+                <param name="device">/dev/arduino_nano</param>
                 <param name="baud_rate">57600</param>
                 <param name="timeout">1000</param>
-                <param name="enc_counts_per_ver">3436</param>
+                <param name="enc_counts_per_rev">616</param>
+            </hardware>
+            <joint name="left_wheel_joint">
+                <command_interface name="velocity">
+                    <param name="min">-0.2</param>
+                    <param name="max">0.2</param>
+                </command_interface>
+                <state_interface name="velocity"/>
+                <state_interface name="position"/>
+            </joint>
+            <joint name="right_wheel_joint">
+                <command_interface name="velocity">
+                    <param name="min">-0.2</param>
+                    <param name="max">0.2</param>
+                </command_interface>
+                <state_interface name="velocity"/>
+                <state_interface name="position"/>
+            </joint>
+        </ros2_control>
+        <!-- <ros2_control name='MPU6050' type='sensor'>
+            <hardware>
+                <plugin>mpu6050_imu_broadcaster/MPU6050Hardware</plugin>
+                <param name='sensor_name'>mpu6050</param>
+                <param name='frame_id'>imu_link</param>
+            </hardware>
+            <sensor name='mpu6050'>
+                <state_interface name='orientation.x'/>
+                <state_interface name='orientation.y'/>
+                <state_interface name='orientation.z'/>
+                <state_interface name='orientation.w'/>
+                <state_interface name='angular_velocity.x'/>
+                <state_interface name='angular_velocity.y'/>
+                <state_interface name='angular_velocity.z'/>
+                <state_interface name='linear_acceleration.x'/>
+                <state_interface name='linear_acceleration.y'/>
+                <state_interface name='linear_acceleration.z'/>
+            </sensor>
+        </ros2_control>         -->
+    </xacro:unless>
+    <xacro:if value="$(arg sim_mode)">
+        <ros2_control name="GazeboSystem" type="system">
+            <hardware>
+                <plugin>gazebo_ros2_control/GazeboSystem</plugin>
             </hardware>
             <joint name="left_wheel_joint">
@@ -26,23 +68,6 @@
                     <param name="max">10</param>
                 </command_interface>
-            </joint>
-        </ros2_control>
-    </xacro:unless>
-    <xacro:if value="$(arg sim_node)">
-        <ros2_control name="GazeboSystem" type="system">
-            <hardware>
-                <plugin>gazebo_ros2_control/GazeboSystem</plugin>
-            </hardware>
-            <joint name="left_wheel_joint">
-                <command_interface name="velocity">
-                    <param name="min">-10</param>
-                    <param name="max">10</param>
-                </command_interface>
-            </joint>
-            <joint name="right_wheel_joint">
-                <command_interface name="velocity">
-                    <param name="min">-10</param>
-                    <param name="max">10</param>
-                </command_interface>
+                <state_interface name="velocity"/>
+                <state_interface name="position"/>
             </joint>
         </ros2_control>
@@ -50,6 +75,6 @@
     <gazebo>
         <plugin name="gazebo_ros2_control" filename="libgazebo_ros2_control.so">
-            <parameter>$(find myfirstbot)/config/my_controller.yaml</parameter>
-            <parameter>$(find myfirstbot)/config/gaz_ros2_ctl_use_sim.yaml</parameter>
+            <parameters>$(find nbt_bot)/config/my_controllers.yaml</parameters>
+            <parameters>$(find nbt_bot)/config/gaz_ros2_ctl_use_sim.yaml</parameters>
         </plugin>
     </gazebo>
